Commit message: added tcp link added control level constraints to arm ros2_controller , verified everything with sim launch (gazebo ros2 control + moveit)

File: src/sorting_arm_description/urdf/sorting_arm.xacro (robot description, xacro)
@@ -27,3 +27,9 @@
     <origin xyz="0 0 0" rpy="0 0 0"/>
   </xacro:robotiq_gripper>
+  <link name="$(arg tf_prefix)tcp"/>
+  <joint name="$(arg tf_prefix)tcp_joint" type="fixed">
+    <parent link="$(arg tf_prefix)robotiq_85_base_link"/>
+    <child link="$(arg tf_prefix)tcp"/>
+    <origin xyz="0 0 0.16" rpy="0 0 0"/>
+  </joint>
 </robot>

File: src/sorting_arm_moveit/config/sorting_arm.urdf.xacro (robot description, xacro)
@@ -1,9 +1,4 @@
 <?xml version="1.0"?>
 <robot xmlns:xacro="http://www.ros.org/wiki/xacro" name="sorting_arm">
-    <xacro:arg name="initial_positions_file" default="initial_positions.yaml" />
-    <!-- Import sorting_arm urdf file -->
-    <xacro:include filename="$(find sorting_arm_description)/urdf/sorting_arm.urdf.xacro" />
-    <!-- Import control_xacro -->
-    <xacro:include filename="sorting_arm.ros2_control.xacro" />
-    <xacro:sorting_arm_ros2_control name="FakeSystem" initial_positions_file="$(arg initial_positions_file)"/>
+    <xacro:include filename="$(find sorting_arm_description)/urdf/sorting_arm.mock.urdf.xacro"/>
 </robot>

Commit message: rebased world to z=0.0 and shifted everything up

File: src/sorting_arm_description/urdf/sorting_arm.xacro (robot description, xacro)
@@ -18,5 +18,5 @@
     physical_parameters_file="$(arg physical_params)"
     visual_parameters_file="$(arg visual_params)">
-    <origin xyz="0 0 0" rpy="0 0 0"/>
+    <origin xyz="0 0 0.500" rpy="0 0 0"/>
   </xacro:ur_robot>
   <xacro:ur_to_robotiq prefix="$(arg tf_prefix)" parent="$(arg tf_prefix)tool0" child="$(arg tf_prefix)robotiq_85_mount_link"/>

Commit message: feat: add MoveIt-based skills framework and custom interfaces
Changes:

1. Created sorting_arm_skills pkg to use moveit api to do pick place as
   actions , added pick place and home as action servers as they are
long running tasks and should have the feature to cancel from outside
and get constant feedback until its executed , action client for
GripperCommand as plan and execute doesnt work on gripper on all cases ,
scenemanager to construct the planning scene with boxes and table and
main skill orchestrator node which launches all the servers , input
given from cmd line for now

2. Created sorting_arm_interfaces for custom home pick and place actions
   , detected object msg and skillresult msg and a service to sync
objects in the planning scene

3. Fixed simulation launch to launch rviz without a seperate launch file
   as we always intended , but need to check ci for that most likely
will fail

4. Added Home pose as a named target by giving joint angles and creating
   a home pose in srdf

Verification:
Home action tested , sync service working , pick action is failing as it
is colliding with the table.

Future:

Fix the colliding for pick and place actions and complete verification
step
Correct headless sim launch for CI needs to be created seperately

File: src/sorting_arm_description/urdf/sorting_arm.xacro (robot description, xacro)
@@ -10,13 +10,39 @@
   <xacro:include filename="robotiq_2f_85/robotiq_2f_85_macro.urdf.xacro"/>
   <link name="world"/>
+  <!-- pedestal raises the shoulder above the tabletop so grasp poses dont fold the elbow -->
+  <!-- collision is 4mm short of the tabletop on purpose, we cant ACM a runtime CollisionObject -->
+  <joint name="$(arg tf_prefix)pedestal_joint" type="fixed">
+    <parent link="world"/>
+    <child link="$(arg tf_prefix)pedestal"/>
+    <origin xyz="0 0 0.500" rpy="0 0 0"/>
+  </joint>
+  <link name="$(arg tf_prefix)pedestal">
+    <visual>
+      <origin xyz="0 0 0.100" rpy="0 0 0"/>
+      <geometry>
+        <box size="0.16 0.16 0.200"/>
+      </geometry>
+    </visual>
+    <collision>
+      <origin xyz="0 0 0.102" rpy="0 0 0"/>
+      <geometry>
+        <box size="0.16 0.16 0.196"/>
+      </geometry>
+    </collision>
+    <inertial>
+      <mass value="5.0"/>
+      <origin xyz="0 0 0.100" rpy="0 0 0"/>
+      <inertia ixx="0.02" ixy="0.0" ixz="0.0" iyy="0.02" iyz="0.0" izz="0.02"/>
+    </inertial>
+  </link>
   <xacro:ur_robot
     name="ur5e"
     tf_prefix="$(arg tf_prefix)"
-    parent="world"
+    parent="$(arg tf_prefix)pedestal"
     joint_limits_parameters_file="$(arg joint_limit_params)"
     kinematics_parameters_file="$(arg kinematics_params)"
     physical_parameters_file="$(arg physical_params)"
     visual_parameters_file="$(arg visual_params)">
-    <origin xyz="0 0 0.500" rpy="0 0 0"/>
+    <origin xyz="0 0 0.200" rpy="0 0 0"/>
   </xacro:ur_robot>
   <xacro:ur_to_robotiq prefix="$(arg tf_prefix)" parent="$(arg tf_prefix)tool0" child="$(arg tf_prefix)robotiq_85_mount_link"/>
