Commit message: feat(camera): add simulated wrist RGB-D camera(through mount) with gazebo support and regenerated collsion matrix

File: src/sorting_arm_description/urdf/sorting_arm.sim.urdf.xacro (robot description, xacro)
@@ -4,3 +4,31 @@
   <xacro:include filename="sorting_arm.xacro"/>
   <xacro:include filename="sorting_arm.gazebo_ros2_control.xacro"/>
+  <gazebo reference="$(arg tf_prefix)camera_link">
+    <sensor name="camera" type="rgbd_camera">
+      <camera>
+        <horizontal_fov>1.5708</horizontal_fov>
+        <image>
+          <width>640</width>
+          <height>480</height>
+          <format>R8G8B8</format>
+        </image>
+        <clip>
+          <near>0.01</near>
+          <far>15</far>
+        </clip>
+        <noise>
+          <type>gaussian</type>
+          <mean>0.0</mean>
+          <stddev>0.007</stddev>
+        </noise>
+        <optical_frame_id>$(arg tf_prefix)camera_link_optical</optical_frame_id>
+        <camera_info_topic>/camera/camera_info</camera_info_topic>
+      </camera>
+      <always_on>true</always_on>
+      <update_rate>20</update_rate>
+      <visualize>true</visualize>
+      <topic>camera</topic>
+      <gz_frame_id>$(arg tf_prefix)camera_link_optical</gz_frame_id>
+    </sensor>
+  </gazebo>
 </robot>

File: src/sorting_arm_description/urdf/sorting_arm.xacro (robot description, xacro)
@@ -53,4 +53,59 @@
     <origin xyz="0 0 0" rpy="0 0 0"/>
   </xacro:robotiq_gripper>
+  <link name="$(arg tf_prefix)camera_mount_link">
+    <visual>
+      <origin xyz="0 -0.03 0.015" rpy="2.677945 0 0"/>
+      <geometry>
+        <box size="0.01 0.067082 0.01"/>
+      </geometry>
+      <material name="camera_black">
+        <color rgba="0.02 0.02 0.02 1.0"/>
+      </material>
+    </visual>
+    <collision>
+      <origin xyz="0 -0.03 0.015" rpy="2.677945 0 0"/>
+      <geometry>
+        <box size="0.01 0.067082 0.01"/>
+      </geometry>
+    </collision>
+    <inertial>
+      <mass value="0.01"/>
+      <inertia ixx="0.000003833333" ixy="0" ixz="0" iyy="0.000000166667" iyz="0" izz="0.000003833333"/>
+    </inertial>
+  </link>
+  <joint name="$(arg tf_prefix)camera_mount_joint" type="fixed">
+    <parent link="$(arg tf_prefix)tool0"/>
+    <child link="$(arg tf_prefix)camera_mount_link"/>
+  </joint>
+  <link name="$(arg tf_prefix)camera_link">
+    <visual>
+      <geometry>
+        <box size="0.035 0.025 0.025"/>
+      </geometry>
+      <material name="camera_black">
+        <color rgba="0.02 0.02 0.02 1.0"/>
+      </material>
+    </visual>
+    <collision>
+      <geometry>
+        <box size="0.035 0.025 0.025"/>
+      </geometry>
+    </collision>
+    <inertial>
+      <mass value="0.02"/>
+      <inertia ixx="0.000002083333" ixy="0" ixz="0" iyy="0.000003083333" iyz="0" izz="0.000003083333"/>
+    </inertial>
+  </link>
+  <joint name="$(arg tf_prefix)camera_joint" type="fixed">
+    <parent link="$(arg tf_prefix)camera_mount_link"/>
+    <child link="$(arg tf_prefix)camera_link"/>
+    <origin xyz="0 -0.06 0.03" rpy="0 ${-pi/2} 0"/>
+  </joint>
+  <link name="$(arg tf_prefix)camera_link_optical"/>
+  <joint name="$(arg tf_prefix)camera_optical_joint" type="fixed">
+    <origin xyz="0 0 0" rpy="${-pi/2} 0 ${-pi/2}"/>
+    <parent link="$(arg tf_prefix)camera_link"/>
+    <child link="$(arg tf_prefix)camera_link_optical"/>
+  </joint>
   <link name="$(arg tf_prefix)tcp"/>
   <joint name="$(arg tf_prefix)tcp_joint" type="fixed">
