Commit message: fix: remove unresolved merge conflict markers from shared-worktree collision
  A concurrent session's stash pop collided with this branch's already-merged
  gripper fix across six files, leaving literal <<<<<<< markers in compiled
  C++ and a duplicate gripper joint block in the ros2_control xacro — CI
  caught it at the build step. Restored all six files to match what's
  actually verified and merged on main.

File: src/sorting_arm_description/urdf/sorting_arm.gazebo_ros2_control.xacro (robot description, xacro)
@@ -41,34 +41,9 @@
             <state_interface name="effort"/>
         </joint>
-<<<<<<< Updated upstream
         <!-- dart's installed plugin has zero mimic feature symbols (checked with nm -D),
              so gz_ros2_control's own control-cycle mimic drive is the followers' only
              enforcer - nothing native competes with it, unlike under bullet_featherstone -->
-=======
-        <!-- we expose follower states for diagnosis but disable ros2_control mimic parsing so
-             Harmonic's native sdf mimic remains the only drive: docs/rca/gripper-grasp-instability.md -->
->>>>>>> Stashed changes
         <joint name="robotiq_85_left_knuckle_joint">
             <command_interface name="position"/>
-            <state_interface name="position"/>
-            <state_interface name="velocity"/>
-        </joint>
-        <joint name="robotiq_85_right_knuckle_joint" mimic="false">
-            <state_interface name="position"/>
-            <state_interface name="velocity"/>
-        </joint>
-        <joint name="robotiq_85_left_inner_knuckle_joint" mimic="false">
-            <state_interface name="position"/>
-            <state_interface name="velocity"/>
-        </joint>
-        <joint name="robotiq_85_right_inner_knuckle_joint" mimic="false">
-            <state_interface name="position"/>
-            <state_interface name="velocity"/>
-        </joint>
-        <joint name="robotiq_85_left_finger_tip_joint" mimic="false">
-            <state_interface name="position"/>
-            <state_interface name="velocity"/>
-        </joint>
-        <joint name="robotiq_85_right_finger_tip_joint" mimic="false">
             <state_interface name="position"/>
             <state_interface name="velocity"/>

Commit message: feat: add wrist-camera perception and integrated bringup
Added perception pkg with wrist cam RGB -D perception via service
Created ObjectDetection service
Implemented perception failure handling

File: src/sorting_arm_description/urdf/sorting_arm.gazebo_ros2_control.xacro (robot description, xacro)
@@ -7,5 +7,7 @@
         <joint name="shoulder_pan_joint">
             <command_interface name="position"/>
-            <state_interface name="position"/>
+            <state_interface name="position">
+                <param name="initial_value">${initial_positions['shoulder_pan_joint']}</param>
+            </state_interface>
             <state_interface name="velocity"/>
             <state_interface name="effort"/>
@@ -13,5 +15,7 @@
         <joint name="shoulder_lift_joint">
             <command_interface name="position"/>
-            <state_interface name="position"/>
+            <state_interface name="position">
+                <param name="initial_value">${initial_positions['shoulder_lift_joint']}</param>
+            </state_interface>
             <state_interface name="velocity"/>
             <state_interface name="effort"/>
@@ -19,5 +23,7 @@
         <joint name="elbow_joint">
             <command_interface name="position"/>
-            <state_interface name="position"/>
+            <state_interface name="position">
+                <param name="initial_value">${initial_positions['elbow_joint']}</param>
+            </state_interface>
             <state_interface name="velocity"/>
             <state_interface name="effort"/>
@@ -25,5 +31,7 @@
         <joint name="wrist_1_joint">
             <command_interface name="position"/>
-            <state_interface name="position"/>
+            <state_interface name="position">
+                <param name="initial_value">${initial_positions['wrist_1_joint']}</param>
+            </state_interface>
             <state_interface name="velocity"/>
             <state_interface name="effort"/>
@@ -31,5 +39,7 @@
         <joint name="wrist_2_joint">
             <command_interface name="position"/>
-            <state_interface name="position"/>
+            <state_interface name="position">
+                <param name="initial_value">${initial_positions['wrist_2_joint']}</param>
+            </state_interface>
             <state_interface name="velocity"/>
             <state_interface name="effort"/>
@@ -37,5 +47,7 @@
         <joint name="wrist_3_joint">
             <command_interface name="position"/>
-            <state_interface name="position"/>
+            <state_interface name="position">
+                <param name="initial_value">${initial_positions['wrist_3_joint']}</param>
+            </state_interface>
             <state_interface name="velocity"/>
             <state_interface name="effort"/>
@@ -46,5 +58,7 @@
         <joint name="robotiq_85_left_knuckle_joint">
             <command_interface name="position"/>
-            <state_interface name="position"/>
+            <state_interface name="position">
+                <param name="initial_value">${initial_positions['robotiq_85_left_knuckle_joint']}</param>
+            </state_interface>
             <state_interface name="velocity"/>
         </joint>

File: src/sorting_arm_description/urdf/sorting_arm.mock.urdf.xacro (robot description, xacro)
@@ -1,4 +1,9 @@
 <?xml version="1.0"?>
 <robot xmlns:xacro="http://wiki.ros.org/xacro" name="sorting_arm">
+  <xacro:arg name="initial_positions_file"
+             default="$(find sorting_arm_description)/config/initial_positions.yaml"/>
+  <xacro:property name="initial_positions_file" value="$(arg initial_positions_file)"/>
+  <xacro:property name="initial_positions"
+                  value="${xacro.load_yaml(initial_positions_file)['initial_positions']}"/>
   <xacro:include filename="sorting_arm.xacro"/>
   <xacro:include filename="sorting_arm.ros2_control.xacro"/>

File: src/sorting_arm_description/urdf/sorting_arm.ros2_control.xacro (robot description, xacro)
@@ -12,5 +12,5 @@
             <command_interface name="position"/>
             <state_interface name="position">
-                <param name="initial_value">0.0</param>
+                <param name="initial_value">${initial_positions['shoulder_pan_joint']}</param>
             </state_interface>
             <state_interface name="velocity"/>
@@ -19,5 +19,5 @@
             <command_interface name="position"/>
             <state_interface name="position">
-                <param name="initial_value">0.0</param>
+                <param name="initial_value">${initial_positions['shoulder_lift_joint']}</param>
             </state_interface>
             <state_interface name="velocity"/>
@@ -26,5 +26,5 @@
             <command_interface name="position"/>
             <state_interface name="position">
-                <param name="initial_value">0.0</param>
+                <param name="initial_value">${initial_positions['elbow_joint']}</param>
             </state_interface>
             <state_interface name="velocity"/>
@@ -33,5 +33,5 @@
             <command_interface name="position"/>
             <state_interface name="position">
-                <param name="initial_value">0.0</param>
+                <param name="initial_value">${initial_positions['wrist_1_joint']}</param>
             </state_interface>
             <state_interface name="velocity"/>
@@ -40,5 +40,5 @@
             <command_interface name="position"/>
             <state_interface name="position">
-                <param name="initial_value">0.0</param>
+                <param name="initial_value">${initial_positions['wrist_2_joint']}</param>
             </state_interface>
             <state_interface name="velocity"/>
@@ -47,5 +47,5 @@
             <command_interface name="position"/>
             <state_interface name="position">
-                <param name="initial_value">0.0</param>
+                <param name="initial_value">${initial_positions['wrist_3_joint']}</param>
             </state_interface>
             <state_interface name="velocity"/>
@@ -55,5 +55,5 @@
             <command_interface name="position"/>
             <state_interface name="position">
-                <param name="initial_value">0.0</param>
+                <param name="initial_value">${initial_positions['robotiq_85_left_knuckle_joint']}</param>
             </state_interface>
             <state_interface name="velocity"/>

File: src/sorting_arm_description/urdf/sorting_arm.sim.urdf.xacro (robot description, xacro)
@@ -2,4 +2,9 @@
 <robot xmlns:xacro="http://wiki.ros.org/xacro" name="sorting_arm">
   <xacro:arg name="controllers_file" default=""/>
+  <xacro:arg name="initial_positions_file"
+             default="$(find sorting_arm_description)/config/initial_positions.yaml"/>
+  <xacro:property name="initial_positions_file" value="$(arg initial_positions_file)"/>
+  <xacro:property name="initial_positions"
+                  value="${xacro.load_yaml(initial_positions_file)['initial_positions']}"/>
   <xacro:include filename="sorting_arm.xacro"/>
   <xacro:include filename="sorting_arm.gazebo_ros2_control.xacro"/>
@@ -9,17 +14,12 @@
         <horizontal_fov>1.5708</horizontal_fov>
         <image>
-          <width>640</width>
-          <height>480</height>
+          <width>1280</width>
+          <height>960</height>
           <format>R8G8B8</format>
         </image>
         <clip>
-          <near>0.01</near>
-          <far>15</far>
+          <near>0.05</near>
+          <far>2.0</far>
         </clip>
-        <noise>
-          <type>gaussian</type>
-          <mean>0.0</mean>
-          <stddev>0.007</stddev>
-        </noise>
         <optical_frame_id>$(arg tf_prefix)camera_link_optical</optical_frame_id>
         <camera_info_topic>/camera/camera_info</camera_info_topic>

File: src/sorting_arm_description/urdf/sorting_arm.xacro (robot description, xacro)
@@ -55,5 +55,5 @@
   <link name="$(arg tf_prefix)camera_mount_link">
     <visual>
-      <origin xyz="0 -0.03 0.015" rpy="2.677945 0 0"/>
+      <origin xyz="0 -0.03 0.015" rpy="-0.463648 0 0"/>
       <geometry>
         <box size="0.01 0.067082 0.01"/>
@@ -64,5 +64,5 @@
     </visual>
     <collision>
-      <origin xyz="0 -0.03 0.015" rpy="2.677945 0 0"/>
+      <origin xyz="0 -0.03 0.015" rpy="-0.463648 0 0"/>
       <geometry>
         <box size="0.01 0.067082 0.01"/>
@@ -70,4 +70,5 @@
     </collision>
     <inertial>
+      <origin xyz="0 -0.03 0.015" rpy="-0.463648 0 0"/>
       <mass value="0.01"/>
       <inertia ixx="0.000003833333" ixy="0" ixz="0" iyy="0.000000166667" iyz="0" izz="0.000003833333"/>
