Commit message: simplified includes in urdf's created and tested bringup pkg to bringup moveit with demo.launch

File: src/sorting_arm_description/urdf/robotiq_2f_85/robotiq_2f_85_macro.urdf.xacro (robot description, xacro)
@@ -5,36 +5,5 @@
         prefix
         parent
-        *origin
-        sim_ignition:=false
-        sim_isaac:=false
-        isaac_joint_commands:=/isaac_joint_commands
-        isaac_joint_states:=/isaac_joint_states
-        use_fake_hardware:=false
-        mock_sensor_commands:=false
-        include_ros2_control:=true
-        com_port:=/dev/ttyUSB0
-        gripper_speed_multiplier:=1.0
-        gripper_force_multiplier:=0.5
-        gripper_max_speed:=0.150
-        gripper_max_force:=235.0
-        gripper_closed_position:=0.7929">
-        <!-- if we are simulating or directly communicating with the gripper we need a ros2 control instance -->
-        <xacro:if value="${include_ros2_control}">
-            <xacro:include filename="$(find sorting_arm_description)/urdf/robotiq_2f_85/2f_85.ros2_control.xacro" />
-            <xacro:robotiq_gripper_ros2_control
-                name="${name}" prefix="${prefix}"
-                sim_ignition="${sim_ignition}"
-                sim_isaac="${sim_isaac}"
-                isaac_joint_commands="${isaac_joint_commands}"
-                isaac_joint_states="${isaac_joint_states}"
-                use_fake_hardware="${use_fake_hardware}"
-                mock_sensor_commands="${mock_sensor_commands}"
-                com_port="${com_port}"
-                gripper_speed_multiplier="${gripper_speed_multiplier}"
-                gripper_force_multiplier="${gripper_force_multiplier}"
-                gripper_max_speed="${gripper_max_speed}"
-                gripper_max_force="${gripper_max_force}"
-                gripper_closed_position="${gripper_closed_position}"/>
-        </xacro:if>
+        *origin">
         <link name="${prefix}robotiq_85_base_link">
             <visual>

File: src/sorting_arm_description/urdf/sorting_arm.ros2_control.xacro (robot description, xacro)
@@ -1,56 +1,53 @@
 <?xml version="1.0"?>
 <robot xmlns:xacro="http://www.ros.org/wiki/xacro">
-    <xacro:macro name="sorting_arm_ros2_control" params="name initial_positions_file">
-        <xacro:property name="initial_positions" value="${xacro.load_yaml(initial_positions_file)['initial_positions']}"/>
-        <ros2_control name="${name}" type="system">
-            <hardware>
-                <!-- By default, set up controllers for simulation. This won't work on real hardware -->
-                <plugin>mock_components/GenericSystem</plugin>
-            </hardware>
-            <joint name="shoulder_pan_joint">
-                <command_interface name="position"/>
-                <state_interface name="position">
-                  <param name="initial_value">${initial_positions['shoulder_pan_joint']}</param>
-                </state_interface>
-            </joint>
-            <joint name="shoulder_lift_joint">
-                <command_interface name="position"/>
-                <state_interface name="position">
-                  <param name="initial_value">${initial_positions['shoulder_lift_joint']}</param>
-                </state_interface>
-            </joint>
-            <joint name="elbow_joint">
-                <command_interface name="position"/>
-                <state_interface name="position">
-                  <param name="initial_value">${initial_positions['elbow_joint']}</param>
-                </state_interface>
-            </joint>
-            <joint name="wrist_1_joint">
-                <command_interface name="position"/>
-                <state_interface name="position">
-                  <param name="initial_value">${initial_positions['wrist_1_joint']}</param>
-                </state_interface>
-            </joint>
-            <joint name="wrist_2_joint">
-                <command_interface name="position"/>
-                <state_interface name="position">
-                  <param name="initial_value">${initial_positions['wrist_2_joint']}</param>
-                </state_interface>
-            </joint>
-            <joint name="wrist_3_joint">
-                <command_interface name="position"/>
-                <state_interface name="position">
-                  <param name="initial_value">${initial_positions['wrist_3_joint']}</param>
-                </state_interface>
-            </joint>
-            <!-- the gripper action controller claims velocity state too, without it the controller never activates -->
-            <joint name="robotiq_85_left_knuckle_joint">
-                <command_interface name="position"/>
-                <state_interface name="position">
-                  <param name="initial_value">${initial_positions['robotiq_85_left_knuckle_joint']}</param>
-                </state_interface>
-                <state_interface name="velocity"/>
-            </joint>
-        </ros2_control>
-    </xacro:macro>
+    <ros2_control name="sorting_arm" type="system">
+        <hardware>
+            <!-- By default, set up controllers for simulation. This won't work on real hardware -->
+            <plugin>mock_components/GenericSystem</plugin>
+        </hardware>
+        <joint name="shoulder_pan_joint">
+            <command_interface name="position"/>
+            <state_interface name="position">
+                <param name="initial_value">0.0</param>
+            </state_interface>
+        </joint>
+        <joint name="shoulder_lift_joint">
+            <command_interface name="position"/>
+            <state_interface name="position">
+                <param name="initial_value">0.0</param>
+            </state_interface>
+        </joint>
+        <joint name="elbow_joint">
+            <command_interface name="position"/>
+            <state_interface name="position">
+                <param name="initial_value">0.0</param>
+            </state_interface>
+        </joint>
+        <joint name="wrist_1_joint">
+            <command_interface name="position"/>
+            <state_interface name="position">
+                <param name="initial_value">0.0</param>
+            </state_interface>
+        </joint>
+        <joint name="wrist_2_joint">
+            <command_interface name="position"/>
+            <state_interface name="position">
+                <param name="initial_value">0.0</param>
+            </state_interface>
+        </joint>
+        <joint name="wrist_3_joint">
+            <command_interface name="position"/>
+            <state_interface name="position">
+                <param name="initial_value">0.0</param>
+            </state_interface>
+        </joint>
+        <!-- the gripper action controller claims velocity state too, without it the controller never activates -->
+        <joint name="robotiq_85_left_knuckle_joint">
+            <command_interface name="position"/>
+            <state_interface name="position">
+                <param name="initial_value">0.0</param>
+            </state_interface>
+            <state_interface name="velocity"/>
+        </joint>
+    </ros2_control>
 </robot>

File: src/sorting_arm_description/urdf/sorting_arm.urdf.xacro (robot description, xacro)
@@ -1,31 +1,6 @@
 <?xml version="1.0"?>
 <robot xmlns:xacro="http://wiki.ros.org/xacro" name="sorting_arm">
-  <xacro:arg name="tf_prefix" default=""/>
-  <xacro:arg name="joint_limit_params" default="$(find sorting_arm_description)/config/joint_limits.yaml"/>
-  <xacro:arg name="kinematics_params" default="$(find sorting_arm_description)/config/default_kinematics.yaml"/>
-  <xacro:arg name="physical_params" default="$(find sorting_arm_description)/config/physical_parameters.yaml"/>
-  <xacro:arg name="visual_params" default="$(find sorting_arm_description)/config/visual_parameters.yaml"/>
-  <xacro:include filename="$(find sorting_arm_description)/urdf/ur5e/ur_macro.xacro"/>
-  <xacro:include filename="$(find sorting_arm_description)/urdf/robotiq_2f_85/ur_to_robotiq_adapter.urdf.xacro"/>
-  <xacro:include filename="$(find sorting_arm_description)/urdf/robotiq_2f_85/robotiq_2f_85_macro.urdf.xacro"/>
-  <link name="world"/>
-  <xacro:ur_robot
-    name="ur5e"
-    tf_prefix="$(arg tf_prefix)"
-    parent="world"
-    joint_limits_parameters_file="$(arg joint_limit_params)"
-    kinematics_parameters_file="$(arg kinematics_params)"
-    physical_parameters_file="$(arg physical_params)"
-    visual_parameters_file="$(arg visual_params)"
-    generate_ros2_control_tag="false">
-    <origin xyz="0 0 0" rpy="0 0 0"/>
-  </xacro:ur_robot>
-  <xacro:ur_to_robotiq prefix="$(arg tf_prefix)" parent="$(arg tf_prefix)tool0" child="$(arg tf_prefix)robotiq_85_mount_link"/>
-  <xacro:robotiq_gripper
-    name="robotiq_2f_85"
-    prefix="$(arg tf_prefix)"
-    parent="$(arg tf_prefix)robotiq_85_mount_link"
-    include_ros2_control="false">
-    <origin xyz="0 0 0" rpy="0 0 0"/>
-  </xacro:robotiq_gripper>
+  <xacro:include filename="sorting_arm.xacro"/>
+  <!-- Ros2 control -->
+  <xacro:include filename="sorting_arm.ros2_control.xacro"/>
 </robot>

File: src/sorting_arm_description/urdf/ur5e/ur_macro.xacro (robot description, xacro)
@@ -42,6 +42,6 @@
      - Muhammad Asif Rana
   -->
-  <xacro:include filename="$(find sorting_arm_description)/urdf/ur5e/inc/ur_transmissions.xacro" />
-  <xacro:include filename="$(find sorting_arm_description)/urdf/ur5e/inc/ur_common.xacro" />
+  <xacro:include filename="inc/ur_transmissions.xacro" />
+  <xacro:include filename="inc/ur_common.xacro" />
   <xacro:macro name="ur_robot" params="
     name
@@ -53,13 +53,9 @@
     physical_parameters_file
     visual_parameters_file
-    generate_ros2_control_tag:=true
     safety_limits:=false
     safety_pos_margin:=0.15
     safety_k_position:=20
-    use_fake_hardware:=false
-    fake_sensor_commands:=false
     sim_gazebo:=false
-    sim_ignition:=false
-    initial_positions:=${dict(shoulder_pan_joint=0.0,shoulder_lift_joint=-1.57,elbow_joint=0.0,wrist_1_joint=-1.57,wrist_2_joint=0.0,wrist_3_joint=0.0)}"
+    sim_ignition:=false"
     >
     <!-- Load configuration data from the provided .yaml files -->
@@ -70,18 +66,4 @@
       visual_parameters_file="${visual_parameters_file}"
       force_abs_paths="${sim_gazebo or sim_ignition}"/>
-    <xacro:if value="${generate_ros2_control_tag}">
-      <!-- ros2 control include -->
-      <xacro:include filename="$(find sorting_arm_description)/urdf/ur5e/ur.ros2_control.xacro" />
-      <!-- ros2 control instance -->
-      <xacro:ur_ros2_control
-        name="${name}"
-        use_fake_hardware="${use_fake_hardware}"
-        initial_positions="${initial_positions}"
-        fake_sensor_commands="${fake_sensor_commands}"
-        sim_gazebo="${sim_gazebo}"
-        sim_ignition="${sim_ignition}"
-        tf_prefix="${tf_prefix}"
-        />
-    </xacro:if>
     <!-- Add URDF transmission elements (for ros_control) -->
     <!--<xacro:ur_arm_transmission prefix="${prefix}" hw_interface="${transmission_hw_interface}" />-->

Commit message: git commit -m "fix(gripper): stabilize grasping and verify object capture
Switch the simulation physics engine from Bullet Featherstone to DART.
Bullet caused the gripper fingers to move asymmetrically, while DART
produced stable and symmetric finger motion.

Replace the fixed 0.8 rad close target with a target calculated from the
object width. This prevents the gripper from continuously driving toward
its mechanical limit after contacting an object.

Verify the grasp using the measured jaw gap and fingertip symmetry from
/joint_states instead of relying only on the controller's stalled flag.
The same measurements are checked again after lifting to confirm the
object is still held.

Verified with red_box_1: /pick completes successfully through grasp,
attach, retreat, and hold verification."

File: src/sorting_arm_description/urdf/robotiq_2f_85/robotiq_2f_85_macro.urdf.xacro (robot description, xacro)
@@ -194,6 +194,6 @@
             <axis xyz="0 -1 0" />
             <origin xyz="0.0127 0.0 0.06142" rpy="0 0 0" />
+            <limit lower="0.0" upper="0.8" velocity="0.5" effort="50" />
             <mimic joint="${prefix}robotiq_85_left_knuckle_joint" />
-            <limit lower="0.0" upper="0.8" velocity="0.5" effort="50" />
         </joint>
         <joint name="${prefix}robotiq_85_right_inner_knuckle_joint" type="revolute">
@@ -202,6 +202,6 @@
             <axis xyz="0 -1 0" />
             <origin xyz="-0.0127 0.0 0.06142" rpy="0 0 0" />
+            <limit lower="-0.8" upper="0.0" velocity="0.5" effort="50" />
             <mimic joint="${prefix}robotiq_85_left_knuckle_joint" multiplier="-1" />
-            <limit lower="-0.8" upper="0.0" velocity="0.5" effort="50" />
         </joint>
         <joint name="${prefix}robotiq_85_left_finger_tip_joint" type="revolute">
@@ -210,6 +210,6 @@
             <axis xyz="0 -1 0" />
             <origin xyz="0.00563134 0.0 0.04718515" rpy="0 0 0" />
+            <limit lower="-0.8" upper="0.0" velocity="0.5" effort="50" />
             <mimic joint="${prefix}robotiq_85_left_knuckle_joint" multiplier="-1" />
-            <limit lower="-0.8" upper="0.0" velocity="0.5" effort="50" />
         </joint>
         <joint name="${prefix}robotiq_85_right_finger_tip_joint" type="revolute">
@@ -218,16 +218,16 @@
             <axis xyz="0 -1 0" />
             <origin xyz="-0.00563134 0.0 0.04718515" rpy="0 0 0" />
+            <limit lower="0.0" upper="0.8" velocity="0.5" effort="50" />
             <mimic joint="${prefix}robotiq_85_left_knuckle_joint" />
-            <limit lower="0.0" upper="0.8" velocity="0.5" effort="50" />
-        </joint>
-        <!-- sdformat only reads friction from a gazebo reference block, the surface
-             block inside collision never reached the sdf so the pads ran at mu=1 -->
+        </joint>
+        <!-- inline <surface> in a URDF <collision> is not schema, gz sdf drops it silently.
+             this is the form that actually reaches bullet_featherstone -->
         <gazebo reference="${prefix}robotiq_85_left_finger_tip_link">
-            <mu1>100000.0</mu1>
-            <mu2>100000.0</mu2>
+            <mu1>5.0</mu1>
+            <mu2>5.0</mu2>
         </gazebo>
         <gazebo reference="${prefix}robotiq_85_right_finger_tip_link">
-            <mu1>100000.0</mu1>
-            <mu2>100000.0</mu2>
+            <mu1>5.0</mu1>
+            <mu2>5.0</mu2>
         </gazebo>
     </xacro:macro>

File: src/sorting_arm_description/urdf/sorting_arm.gazebo_ros2_control.xacro (robot description, xacro)
@@ -41,4 +41,7 @@
             <state_interface name="effort"/>
         </joint>
+        <!-- dart's installed plugin has zero mimic feature symbols (checked with nm -D),
+             so no native constraint exists to fight gz_ros2_control's own mimic drive -
+             followers stay state-only, but mimic="false" is gone or theyd get no drive at all -->
         <joint name="robotiq_85_left_knuckle_joint">
             <command_interface name="position"/>

Commit message: fix: stabilize gripper grasping and verify object capture (#2)
* fix(skills): make pick grasp failures measurable

  Issue:

  The pick behavior was inconsistent. The gripper sometimes timed out
while
  shaking, sometimes completed the action but dropped the cube during
retreat,
  and sometimes left old close commands running.

  Things we did:

  - Replaced the step-by-step close ladder with one GripperCommand goal.
  - Used the controller's stalled result to detect object contact.
  - Cancelled a gripper goal when the client timeout expires.
  - Enabled allow_stalling and set stall_velocity_threshold to 0.02.
  - Added bounded pre-grasp candidate search.
  - Checked the complete Cartesian descent before moving the robot.
  - Temporarily allowed contact with the target object during grasp
    planning.
  - Used MoveIt's joint limits when retiming Cartesian trajectories.
  - Lowered grasp_offset_m from -0.02 to -0.036 so the pads cover more
    of the cube face.
  - Moved fingertip friction into Gazebo reference blocks so it reaches
    the generated SDF.
  - Added an open RCA with the investigation history and remaining work.

  What worked:

  - The gripper now receives one close goal instead of many overlapping
    goals.
  - One run returned SUCCEEDED with stalled true in about one second.
  - The pick reached attach and retreat without the old simulation-time
    retiming error.
  - Pre-grasp candidate search found a valid candidate after earlier
    candidates
    failed.
  - The complete Cartesian descent executed successfully.
  - The deeper grasp position places about 37 mm of the 40 mm cube face
    between the pads.

  What happened:

  - The cube still fell during retreat.
  - Activating fingertip friction at mu=100000 caused visible contact
    shaking.
  - The latest successful close took about 9.70 seconds, almost reaching
    the
    10-second client timeout.
  - Small timing differences now decide whether close succeeds or
    aborts.
  - This commit records the current investigation baseline. It is not
    the
    completed gripper fix.
  - Current Status is that it is sometimes grasping completing the
    action but dropping the cube sometimes it fails to grasp itself and
    action is aborted.

* git commit -m "fix(gripper): stabilize grasping and verify object capture

Switch the simulation physics engine from Bullet Featherstone to DART.
Bullet caused the gripper fingers to move asymmetrically, while DART
produced stable and symmetric finger motion.

Replace the fixed 0.8 rad close target with a target calculated from the
object width. This prevents the gripper from continuously driving toward
its mechanical limit after contacting an object.

Verify the grasp using the measured jaw gap and fingertip symmetry from
/joint_states instead of relying only on the controller's stalled flag.
The same measurements are checked again after lifting to confirm the
object is still held.

Verified with red_box_1: /pick completes successfully through grasp,
attach, retreat, and hold verification."

File: src/sorting_arm_description/urdf/robotiq_2f_85/robotiq_2f_85_macro.urdf.xacro (robot description, xacro)
@@ -135,22 +135,4 @@
                     <mesh filename="file://$(find sorting_arm_description)/meshes/robotiq_2f_85/collision/2f_85/left_finger_tip.stl" />
                 </geometry>
-                <surface>
-                    <friction>
-                    <ode>
-                        <mu1>100000.0</mu1>
-                        <mu2>100000.0</mu2>
-                    </ode>
-                    </friction>
-                    <contact>
-                    <ode>
-                        <kp>1e+5</kp>
-                        <kd>1</kd>
-                        <soft_cfm>0</soft_cfm>
-                        <soft_erp>0.2</soft_erp>
-                        <minDepth>0.002</minDepth>
-                        <maxVel>0</maxVel>
-                    </ode>
-                    </contact>
-                </surface>
             </collision>
             <inertial>
@@ -170,22 +152,4 @@
                     <mesh filename="file://$(find sorting_arm_description)/meshes/robotiq_2f_85/collision/2f_85/right_finger_tip.stl" />
                 </geometry>
-                <surface>
-                    <friction>
-                    <ode>
-                        <mu1>100000.0</mu1>
-                        <mu2>100000.0</mu2>
-                    </ode>
-                    </friction>
-                    <contact>
-                    <ode>
-                        <kp>1e+5</kp>
-                        <kd>1</kd>
-                        <soft_cfm>0</soft_cfm>
-                        <soft_erp>0.2</soft_erp>
-                        <minDepth>0.002</minDepth>
-                        <maxVel>0</maxVel>
-                    </ode>
-                    </contact>
-                </surface>
             </collision>
             <inertial>
@@ -230,6 +194,6 @@
             <axis xyz="0 -1 0" />
             <origin xyz="0.0127 0.0 0.06142" rpy="0 0 0" />
+            <limit lower="0.0" upper="0.8" velocity="0.5" effort="50" />
             <mimic joint="${prefix}robotiq_85_left_knuckle_joint" />
-            <limit lower="0.0" upper="0.8" velocity="0.5" effort="50" />
         </joint>
         <joint name="${prefix}robotiq_85_right_inner_knuckle_joint" type="revolute">
@@ -238,6 +202,6 @@
             <axis xyz="0 -1 0" />
             <origin xyz="-0.0127 0.0 0.06142" rpy="0 0 0" />
+            <limit lower="-0.8" upper="0.0" velocity="0.5" effort="50" />
             <mimic joint="${prefix}robotiq_85_left_knuckle_joint" multiplier="-1" />
-            <limit lower="-0.8" upper="0.0" velocity="0.5" effort="50" />
         </joint>
         <joint name="${prefix}robotiq_85_left_finger_tip_joint" type="revolute">
@@ -246,6 +210,6 @@
             <axis xyz="0 -1 0" />
             <origin xyz="0.00563134 0.0 0.04718515" rpy="0 0 0" />
+            <limit lower="-0.8" upper="0.0" velocity="0.5" effort="50" />
             <mimic joint="${prefix}robotiq_85_left_knuckle_joint" multiplier="-1" />
-            <limit lower="-0.8" upper="0.0" velocity="0.5" effort="50" />
         </joint>
         <joint name="${prefix}robotiq_85_right_finger_tip_joint" type="revolute">
@@ -254,7 +218,17 @@
             <axis xyz="0 -1 0" />
             <origin xyz="-0.00563134 0.0 0.04718515" rpy="0 0 0" />
+            <limit lower="0.0" upper="0.8" velocity="0.5" effort="50" />
             <mimic joint="${prefix}robotiq_85_left_knuckle_joint" />
-            <limit lower="0.0" upper="0.8" velocity="0.5" effort="50" />
-        </joint>
+        </joint>
+        <!-- inline <surface> in a URDF <collision> is not schema, gz sdf drops it silently.
+             this is the form that actually reaches bullet_featherstone -->
+        <gazebo reference="${prefix}robotiq_85_left_finger_tip_link">
+            <mu1>5.0</mu1>
+            <mu2>5.0</mu2>
+        </gazebo>
+        <gazebo reference="${prefix}robotiq_85_right_finger_tip_link">
+            <mu1>5.0</mu1>
+            <mu2>5.0</mu2>
+        </gazebo>
     </xacro:macro>
 </robot>
