Commit message: chore(gripper): clean up debug residue, add app launch and sequence demo
Removes temporary debugging changes that are no longer needed, including the bag bridge, joint-order changes, and unused stall threshold.

Adds `app.launch.xml` so the full sorting cell can be started with one command.

Adds `sequence_demo` for manually testing the complete pick-and-place flow.

Shortens the grasp debugging document from 1,654 lines to 246 lines.

Also fixes the runtime Dockerfile by copying the missing `sorting_arm_interfaces/package.xml`, allowing `rosdep` to install its dependencies correctly during the image build.

File: src/sorting_arm_description/urdf/robotiq_2f_85/robotiq_2f_85_macro.urdf.xacro (robot description, xacro)
@@ -194,6 +194,6 @@
             <axis xyz="0 -1 0" />
             <origin xyz="0.0127 0.0 0.06142" rpy="0 0 0" />
+            <mimic joint="${prefix}robotiq_85_left_knuckle_joint" />
             <limit lower="0.0" upper="0.8" velocity="0.5" effort="50" />
-            <mimic joint="${prefix}robotiq_85_left_knuckle_joint" />
         </joint>
         <joint name="${prefix}robotiq_85_right_inner_knuckle_joint" type="revolute">
@@ -202,6 +202,6 @@
             <axis xyz="0 -1 0" />
             <origin xyz="-0.0127 0.0 0.06142" rpy="0 0 0" />
+            <mimic joint="${prefix}robotiq_85_left_knuckle_joint" multiplier="-1" />
             <limit lower="-0.8" upper="0.0" velocity="0.5" effort="50" />
-            <mimic joint="${prefix}robotiq_85_left_knuckle_joint" multiplier="-1" />
         </joint>
         <joint name="${prefix}robotiq_85_left_finger_tip_joint" type="revolute">
@@ -210,6 +210,6 @@
             <axis xyz="0 -1 0" />
             <origin xyz="0.00563134 0.0 0.04718515" rpy="0 0 0" />
+            <mimic joint="${prefix}robotiq_85_left_knuckle_joint" multiplier="-1" />
             <limit lower="-0.8" upper="0.0" velocity="0.5" effort="50" />
-            <mimic joint="${prefix}robotiq_85_left_knuckle_joint" multiplier="-1" />
         </joint>
         <joint name="${prefix}robotiq_85_right_finger_tip_joint" type="revolute">
@@ -218,9 +218,10 @@
             <axis xyz="0 -1 0" />
             <origin xyz="-0.00563134 0.0 0.04718515" rpy="0 0 0" />
+            <mimic joint="${prefix}robotiq_85_left_knuckle_joint" />
             <limit lower="0.0" upper="0.8" velocity="0.5" effort="50" />
-            <mimic joint="${prefix}robotiq_85_left_knuckle_joint" />
-        </joint>
-        <!-- inline <surface> in a URDF <collision> is not schema, gz sdf drops it silently.
-             this is the form that actually reaches bullet_featherstone -->
+        </joint>
+        <!-- inline <surface> in a URDF <collision> is invalid schema, gz sdf dropped it
+             silently - this <gazebo> form is what actually reaches the physics engine.
+             mu1/mu2=5.0 matches the box's own friction (sorting_cell.sdf); never A/B tested alone -->
         <gazebo reference="${prefix}robotiq_85_left_finger_tip_link">
             <mu1>5.0</mu1>

File: src/sorting_arm_description/urdf/sorting_arm.gazebo_ros2_control.xacro (robot description, xacro)
@@ -41,9 +41,34 @@
             <state_interface name="effort"/>
         </joint>
+<<<<<<< Updated upstream
         <!-- dart's installed plugin has zero mimic feature symbols (checked with nm -D),
-             so no native constraint exists to fight gz_ros2_control's own mimic drive -
-             followers stay state-only, but mimic="false" is gone or theyd get no drive at all -->
+             so gz_ros2_control's own control-cycle mimic drive is the followers' only
+             enforcer - nothing native competes with it, unlike under bullet_featherstone -->
+=======
+        <!-- we expose follower states for diagnosis but disable ros2_control mimic parsing so
+             Harmonic's native sdf mimic remains the only drive: docs/rca/gripper-grasp-instability.md -->
+>>>>>>> Stashed changes
         <joint name="robotiq_85_left_knuckle_joint">
             <command_interface name="position"/>
+            <state_interface name="position"/>
+            <state_interface name="velocity"/>
+        </joint>
+        <joint name="robotiq_85_right_knuckle_joint" mimic="false">
+            <state_interface name="position"/>
+            <state_interface name="velocity"/>
+        </joint>
+        <joint name="robotiq_85_left_inner_knuckle_joint" mimic="false">
+            <state_interface name="position"/>
+            <state_interface name="velocity"/>
+        </joint>
+        <joint name="robotiq_85_right_inner_knuckle_joint" mimic="false">
+            <state_interface name="position"/>
+            <state_interface name="velocity"/>
+        </joint>
+        <joint name="robotiq_85_left_finger_tip_joint" mimic="false">
+            <state_interface name="position"/>
+            <state_interface name="velocity"/>
+        </joint>
+        <joint name="robotiq_85_right_finger_tip_joint" mimic="false">
             <state_interface name="position"/>
             <state_interface name="velocity"/>
